File: klor-trackball/PCB/konrad_trackball/konrad_trackball.kicad_sch (KiCad schematic)
At the start: 88 parts, among them J1 MJ-4PP-9, J2 Haptic Buzz, J3 lv27, SW1 SW_PUSH-MX_W_LED, SW10 SW_PUSH-MX_W_LED, SW11 SW_PUSH-MX_W_LED, SW12 SW_PUSH-MX_W_LED, SW13 SW_PUSH-MX_W_LED, SW14 SW_PUSH-MX_W_LED, SW15 SW_PUSH-MX_W_LED, SW16 SW_PUSH-MX_W_LED, SW17 SW_PUSH-MX_W_LED, SW18 RotaryEncoder_Switch, SW19 SW_PUSH-MX_W_LED, SW2 SW_PUSH-MX_W_LED, SW20 SW_PUSH-MX_W_LED, SW21 SW_PUSH-MX_W_LED, SW22 SW_PUSH-MX_W_LED, SW3 SW_PUSH-MX_W_LED, SW4 SW_PUSH-MX_W_LED, SW5 SW_PUSH-MX_W_LED, SW6 SW_PUSH-MX_W_LED, SW7 SW_PUSH-MX_W_LED, SW8 SW_PUSH-MX_W_LED, SW9 SW_PUSH-MX_W_LED, U1 ProMicro

Commit message: task3b: implement frozen schematic contract
Parts:
- removed D22: D_Small, KLOR:Diode_SOD123, symbol Device:D_Small
- removed SW22: SW_PUSH-MX_W_LED, KLOR:SK6812MINI_and_cherry_1, symbol KLORlib:SW_PUSH-MX_W_LED
- added J4: PMW3360 Kivipallur, Connector_PinHeader_2.54mm:PinHeader_1x07_P2.54mm_Vertical, symbol Connector_Generic:Conn_01x07
- BZ1, J2, OLED1: now not fitted
Connections:
- net AUDIO: no longer U1.12 (9/B5)
- net GND: now also SW13.1 (DOUT), SW14.3 (DIN), J4.7 (Pin_7)
- net SCL: no longer U1.6 (3/D0/SCL)
- net SDA: no longer U1.5 (2/D1/SDA)
- net VCC: now also J4.6 (Pin_6)
- net RX: no longer names the net of J1.3
- net RX: no longer U1.7 (4/D4)
- new net PMW_CS: J4.1 (Pin_1), U1.12 (9/B5)
- new net PMW_MISO: J4.2 (Pin_2), U1.7 (4/D4)
- new net PMW_MOSI: J4.3 (Pin_3), U1.6 (3/D0/SCL)
- new net PMW_SCK: J4.4 (Pin_4), U1.5 (2/D1/SDA)
- no-connect marks 2 -> 4
