File: klor-trackball/PCB/konrad_trackball/konrad_trackball.kicad_pcb (KiCad board)
At the start: 2 copper layers, 160 x 118.2 mm, 89 parts, among them J1 MJ-4PP-9, J2 Haptic Buzz, J3 lv27, SW1 SW_PUSH-MX_W_LED, SW10 SW_PUSH-MX_W_LED, SW11 SW_PUSH-MX_W_LED, SW12 SW_PUSH-MX_W_LED, SW13 SW_PUSH-MX_W_LED, SW14 SW_PUSH-MX_W_LED, SW15 SW_PUSH-MX_W_LED, SW16 SW_PUSH-MX_W_LED, SW17 SW_PUSH-MX_W_LED, SW18 RotaryEncoder_Switch, SW19 SW_PUSH-MX_W_LED, SW2 SW_PUSH-MX_W_LED, SW20 SW_PUSH-MX_W_LED, SW21 SW_PUSH-MX_W_LED, SW22 SW_PUSH-MX_W_LED, SW3 SW_PUSH-MX_W_LED, SW4 SW_PUSH-MX_W_LED, SW5 SW_PUSH-MX_W_LED, SW6 SW_PUSH-MX_W_LED, SW7 SW_PUSH-MX_W_LED, SW8 SW_PUSH-MX_W_LED, SW9 SW_PUSH-MX_W_LED, U1 ProMicro

Commit message: task3c: generate synchronized PCB
Parts:
- removed D22: D_Small, KLOR:Diode_SOD123
- removed SW22: SW_PUSH-MX_W_LED, KLOR:SK6812MINI_and_cherry_1
- added J4: PMW3360 Kivipallur, Connector_PinHeader_2.54mm:PinHeader_1x07_P2.54mm_Vertical, F.Cu at (60.0, 70.0)
Connections:
- J1 pad 3: RX -> (no net)
- SW14 pad 3: Net-(SW14B-DIN) -> Net-(SW13B-DOUT)
- U1 pad 12: AUDIO -> PMW_CS
- U1 pad 5: SDA -> PMW_SCK
- U1 pad 6: SCL -> PMW_MOSI
- U1 pad 7: RX -> PMW_MISO
Routing:
- net RX: track 82.7 -> 0.00 mm, vias 2 -> 0
- net Net-(SW14B-DIN): track 44.2 -> 0.00 mm, vias 2 -> 0
- net col1: track 294.6 -> 259.6 mm, vias 7 -> 6
- net AUDIO: track 103.2 -> 73.0 mm
- net Net-(SW13B-DOUT): track 44.6 -> 70.0 mm, vias 3 -> 4
- net Net-(D22-A): track 22.1 -> 0.00 mm, vias 1 -> 0
- net SDA: track 279.5 -> 258.1 mm
- net row3: track 166.7 -> 145.4 mm
- net SCL: track 260.6 -> 239.7 mm
- net PMW_SCK: track 0.00 -> 17.0 mm
- net PMW_MISO: track 0.00 -> 17.0 mm
- net PMW_CS: track 0.00 -> 17.0 mm
- net PMW_MOSI: track 0.00 -> 17.0 mm
